File: KiCad/miniParMain.kicad_sch (KiCad schematic)
At the start: 35 parts, among them J1 Conn_01x08, J2 USB_C_Receptacle, J4 Conn_01x02_Pin, J5 secondBoard, SW2 SW_Push, U1 AS7341-DLGT, U2 IP4234CZ6, U5 AP7312-1833W6-7, U8 ESP8685, Y2 40MHz

Commit message: PCB revision -> V 1.1
Parts:
- added D3: LED, Diode_SMD:D_0805_2012Metric, symbol Device:LED
- added R13: 5.1K, Resistor_SMD:R_0603_1608Metric, symbol main-rescue:R-
- D1: footprint Diode_SMD:D_SOD-523 -> Diode_SMD:D_SOD-123
- D2: footprint Personal_Library:NF2W757GT-F1 -> Diode_SMD:D_0805_2012Metric
- R2: footprint Resistor_SMD:R_0603_1608Metric_Pad0.98x0.95mm_HandSolder -> Resistor_SMD:R_0603_1608Metric
- SW2: footprint Button_Switch_SMD:SW_SPST_TS-1088-xR025 -> Button_Switch_SMD:SW_SPST_EVQP2_ShortPushTravel_H2.1mm
- U5: footprint Package_TO_SOT_SMD:TSOT-23-6_HandSoldering -> Package_TO_SOT_SMD:TSOT-23-6
Connections:
- net GND: now also R13.1
- net at U8.16 (GPIO10): now also D3.2 (A)
- new net: D3.1 (K), R13.2
- no-connect marks 17 -> 16
Other:
- note added: "Changes 1.0 - 1.1 * 1N4148 package * new status LED - D3 * button footprint change"
